File: Garbage_collector_pcb/STM32.kicad_sch (KiCad schematic)
At the start: 17 parts, among them J2 Conn_ST_STDC14, U3 STM32G431KBTx, Y1 16MHz

Commit message: changement stm
Parts:
- added C12, C13, C14, C18, C20: 100n, Capacitor_SMD:C_0402_1005Metric_Pad0.74x0.62mm_HandSolder, symbol Device:C_Small
- added C15: 10n, Capacitor_SMD:C_0402_1005Metric_Pad0.74x0.62mm_HandSolder, symbol Device:C_Small
- added C16, C19: 1u, Capacitor_SMD:C_0402_1005Metric_Pad0.74x0.62mm_HandSolder, symbol Device:C_Small
- added C17: 4.7u, Capacitor_SMD:C_0402_1005Metric_Pad0.74x0.62mm_HandSolder, symbol Device:C_Small
- added C21, C22: 10pF, Capacitor_SMD:C_0402_1005Metric, symbol Device:C_Small
- added R7: 390, Resistor_THT:R_Array_SIP4, symbol Device:R_Small
- added U2: STM32G431RBTx, Package_QFP:LQFP-64_10x10mm_P0.5mm, symbol MCU_ST_STM32G4:STM32G431RBTx
- added Y2: 16MHz, Crystal:Crystal_SMD_EuroQuartz_MT-4Pin_3.2x2.5mm, symbol Device:Crystal_GND24_Small
Connections:
- net +3.3V: now also C12.2, C13.2, C14.2, C15.2, C16.2, C17.1, C18.2, C19.2, C20.2, U2.1 (VBAT), U2.16 (VDD), U2.28 (VREF+), U2.29 (VDDA), U2.32 (VDD), U2.48 (VDD), U2.64 (VDD)
- net GND: now also C12.1, C13.1, C14.1, C15.1, C16.1, C17.2, C18.1, C19.1, C20.1, C21.2, C22.2, U2.15 (VSS), U2.27 (VSSA), U2.31 (VSS), U2.47 (VSS), U2.63 (VSS), Y2.2 (G), Y2.4 (G)
- net STM32_D+: no longer names the net of U3.22 (PA12)
- net STM32_D-: no longer names the net of U3.21 (PA11)
- new net: C21.1, R7.2, Y2.3
- new net: C22.1, U2.5 (PF0), Y2.1
- new net: R7.1, U2.6 (PF1)
- no-connect marks 17 -> 19
Other:
- moved on the sheet: C10, C3, C4, C5, C6, C7, C8, C9, D1, D2, J2, R3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
