File: Garbage_collector_pcb/STM32.kicad_sch (KiCad schematic)
At the start: 17 parts, among them J2 Conn_ST_STDC14, U3 STM32G431KBTx, Y1 16MHz

Commit message: Ajout de la partie alimentation
Changed lines of the file:
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@@
 	(wire
 		(pts
-			(xy 125.73 87.63) (xy 111.76 87.63)
+			(xy 113.03 87.63) (xy 111.76 87.63)
 		)
 		(stroke
@@
 	(wire
 		(pts
-			(xy 124.46 95.25) (xy 111.76 95.25)
+			(xy 114.3 95.25) (xy 111.76 95.25)
 		)
 		(stroke
@@
 	(wire
 		(pts
-			(xy 125.73 90.17) (xy 111.76 90.17)
+			(xy 113.03 90.17) (xy 111.76 90.17)
 		)
 		(stroke
@@
 	(wire
 		(pts
-			(xy 124.46 92.71) (xy 111.76 92.71)
+			(xy 114.3 92.71) (xy 111.76 92.71)
 		)
 		(stroke
@@
 	)
 	(label "JTMS/SWDIO"
-		(at 124.46 92.71 180)
-		(effects
-			(font
-				(size 1.27 1.27)
-			)
-			(justify right bottom)
+		(at 114.3 92.71 0)
+		(effects
+			(font
+				(size 1.27 1.27)
+			)
+			(justify left bottom)
 		)
 	)
@@
 	)
 	(label "JCLK/SWCLK"
-		(at 124.46 95.25 180)
-		(effects
-			(font
-				(size 1.27 1.27)
-			)
-			(justify right bottom)
+		(at 114.3 95.25 0)
+		(effects
+			(font
+				(size 1.27 1.27)
+			)
+			(justify left bottom)
 		)
 	)
 	(hierarchical_label "STM32_D+"
 		(shape bidirectional)
-		(at 125.73 90.17 0)
+		(at 113.03 90.17 0)
 		(effects
 			(font
@@
 	(hierarchical_label "STM32_D-"
 		(shape bidirectional)
-		(at 125.73 87.63 0)
-		(effects
-			(font
+		(at 113.03 87.63 0)
+		(effects
+			(font

Commit message: seance 24 septembre
Parts:
- removed C10, C9: 10pF, Capacitor_SMD:C_0402_1005Metric, symbol Device:C_Small
- removed C3, C4, C8: 100n, Capacitor_SMD:C_0402_1005Metric, symbol Device:C_Small
- removed C5: 4u7, Capacitor_SMD:C_0402_1005Metric, symbol Device:C_Small
- removed C6: 10n, Capacitor_SMD:C_0402_1005Metric, symbol Device:C_Small
- removed C7: 1u, Capacitor_SMD:C_0402_1005Metric, symbol Device:C_Small
- removed U3: STM32G431KBTx, Package_QFP:LQFP-32_7x7mm_P0.8mm, symbol MCU_ST_STM32G4:STM32G431KBTx
- removed Y1: 16MHz, Crystal:Crystal_SMD_EuroQuartz_MT-4Pin_3.2x2.5mm, symbol Device:Crystal_GND24_Small
- added C12, C13, C14, C18, C20: 100n, Capacitor_SMD:C_0402_1005Metric_Pad0.74x0.62mm_HandSolder, symbol Device:C_Small
- added C15: 10n, Capacitor_SMD:C_0402_1005Metric_Pad0.74x0.62mm_HandSolder, symbol Device:C_Small
- added C16, C19: 1u, Capacitor_SMD:C_0402_1005Metric_Pad0.74x0.62mm_HandSolder, symbol Device:C_Small
- added C17: 4.7u, Capacitor_SMD:C_0402_1005Metric_Pad0.74x0.62mm_HandSolder, symbol Device:C_Small
- added C21, C22: 20pF, Capacitor_SMD:C_0402_1005Metric, symbol Device:C_Small
- added C25: 100n, Capacitor_SMD:C_0402_1005Metric, symbol Device:C_Small
- added C26, C27: 6p8, Capacitor_SMD:C_0402_1005Metric, symbol Device:C_Small
- added R7: 390, Resistor_THT:R_Array_SIP4, symbol Device:R_Small
- added SW2: SW_Push, symbol Kicad:SW_Push
- added U2: STM32G431RBTx, Package_QFP:LQFP-64_10x10mm_P0.5mm, symbol MCU_ST_STM32G4:STM32G431RBTx
- added Y2: 24MHz, Crystal:Crystal_SMD_EuroQuartz_MT-4Pin_3.2x2.5mm, symbol Device:Crystal_GND24_Small
- added Y3: 32KHz, Crystal:Crystal_SMD_EuroQuartz_MT-4Pin_3.2x2.5mm, symbol Device:Crystal_GND24_Small
Connections:
- net +3.3V: now also C12.2, C13.2, C14.2, C15.2, C16.2, C17.1, C18.2, C19.2, C20.2, U2.1 (VBAT), U2.16 (VDD), U2.28 (VREF+), U2.29 (VDDA), U2.32 (VDD), U2.48 (VDD), U2.64 (VDD)
- net GND: now also C12.1, C13.1, C14.1, C15.1, C16.1, C17.2, C18.1, C19.1, C20.1, C21.2, C22.2, C25.2, SW2.2, U2.15 (VSS), U2.27 (VSSA), U2.31 (VSS), U2.47 (VSS), U2.63 (VSS), Y2.2 (G), Y2.4 (G)
- new net: C21.1, R7.2, Y2.3
- new net: C27.1, U2.3 (PC14), Y3.1
- new net: C26.2, C27.2, Y3.2 (G), Y3.4 (G)
- new net: C25.1, SW2.1, U2.7 (PG10)
- new net: C22.1, U2.5 (PF0), Y2.1
- new net: C26.1, U2.4 (PC15), Y3.3
- new net: R7.1, U2.6 (PF1)
- new net I2C1_SCL: U2.60 (PB7)
- new net I2C1_SDA: U2.61 (PB8)
- new net I2C3_SCL: U2.40 (PC8)
- new net I2C3_SDA: U2.41 (PC9)
- no-connect marks 17 -> 2
Other:
- moved on the sheet: D1, D2, J2, R3, R4

Commit message: update schematic
Parts:
- U2: value STM32G431RBTx -> BQ25896RTWR; footprint Package_QFP:LQFP-64_10x10mm_P0.5mm -> Package_DFN_QFN:Texas_RTW_WQFN-24-1EP_4x4mm_P0.5mm_EP2.7x2.7mm; Availability (none) -> In Stock; CREATOR (none) -> NEZY; Check_prices (none) -> https://www.snapeda.com/parts/BQ25896RTWR/Texas+Instruments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; MANUFACTURER (none) -> Texas Instruments; MAXIMUM_PACKAGE_HEIGHT (none) -> 0.80mm; MF (none) -> Texas Instruments; MP (none) -> BQ25896RTWR; PARTREV (none) -> C; Package (none) -> WQFN-24 Texas Instruments; Price (none) -> None; STANDARD (none) -> Manufacturer Recommendations; SnapEDA_Link (none) -> https://www.snapeda.com/parts/BQ25896RTWR/Texas+Instruments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
Connections:
- net +3.3V: no longer U2.1 (VBAT), U2.16 (VDD), U2.28 (VREF+), U2.29 (VDDA), U2.32 (VDD), U2.48 (VDD), U2.64 (VDD)
- net GND: no longer U2.15 (VSS), U2.27 (VSSA), U2.31 (VSS), U2.47 (VSS), U2.63 (VSS)
- net I2C1_SCL: no longer U2.60 (PB7)
- net I2C1_SDA: no longer U2.61 (PB8)
- net I2C3_SCL: no longer U2.40 (PC8)
- net I2C3_SDA: now also U2.6 (SDA); no longer U2.41 (PC9)
- net at C27.1, Y3.1: no longer U2.3 (PC14)
- net at C25.1, SW2.1: no longer U2.7 (PG10)
- net at C22.1, Y2.1: no longer U2.5 (PF0)
- net at U2.13 (BAT): now also U2.14 (BAT)
- net EXP: now reaches U2.17 (PGND)
- net EXP: now also U2.18 (PGND), U2.25 (EXP)
- net at U2.19 (SW): now also U2.20 (SW)
- net at C26.1, Y3.3: no longer U2.4 (PC15)
- net at R7.1: now also U2.1 (VBUS); no longer U2.6 (PF1)
- new net: U2.15 (SYS), U2.16 (SYS)
Changed lines of the file:
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@@
 		(fields_autoplaced yes)
 		(property "Reference" "U2"
-			(at 102.4733 133.35 0)
-			(show_name no)
-			(do_not_autoplace no)
-			(effects
-				(font
-					(size 1.27 1.27)
-				)
-				(justify left)
-			)
-		)
-		(property "Value" "STM32G431RBTx"
-			(at 102.4733 135.89 0)
-			(show_name no)
-			(do_not_autoplace no)
-			(effects
-				(font
-					(size 1.27 1.27)
-				)
-				(justify left)
-			)
-		)
-		(property "Footprint" "Package_QFP:LQFP-64_10x10mm_P0.5mm"
-			(at 82.55 130.81 0)
-			(hide yes)
-			(show_name no)
-			(do_not_autoplace no)
-			(effects
-				(font
-					(size 1.27 1.27)
-				)
-				(justify right)
-			)
-		)
-		(property "Datasheet" "https://www.st.com/resource/en/datasheet/stm32g431rb.pdf"
+			(at 97.79 49.53 0)
+			(show_name no)
+			(do_not_autoplace no)
+			(effects
+				(font
+					(size 1.27 1.27)
+				)
+			)
+		)
+		(property "Value" "BQ25896RTWR"
+			(at 97.79 52.07 0)
+			(show_name no)
+			(do_not_autoplace no)
+			(effects
+				(font
+					(size 1.27 1.27)
+				)
+			)
+		)
+		(property "Footprint" "Package_DFN_QFN:Texas_RTW_WQFN-24-1EP_4x4mm_P0.5mm_EP2.7x2.7mm"
+			(at 89.408 125.73 0)
+			(hide yes)
+			(show_name no)
+			(do_not_autoplace no)
+			(effects
+				(font
+					(size 1.27 1.27)
+				)
+				(justify bottom)
+			)
+		)
+		(property "Datasheet" ""
 			(at 97.79 85.09 0)
 			(hide yes)
@@
 			)
 		)
-		(property "Description" "STMicroelectronics Arm Cortex-M4 MCU, 128KB flash, 32KB RAM, 170 MHz, 1.71-3.6V, 52 GPIO, LQFP64"
+		(property "Description" "I2C 1cell 3A buck battery charger with power path and PSEL"
+			(at 89.408 125.73 0)
+			(hide yes)
+			(show_name no)
+			(do_not_autoplace no)
+			(effects
+				(font
+					(size 1.27 1.27)
+				)
+				(justify bottom)
+			)
+		)
+		(property "MF" "Texas Instruments"
+			(at 83.82 126.746 0)
+			(hide yes)
+			(show_name no)
+			(do_not_autoplace no)
+			(effects
+				(font
+					(size 1.27 1.27)
+				)
+				(justify bottom)
+			)
+		)
+		(property "MAXIMUM_PACKAGE_HEIGHT" "0.80mm"
+			(at 83.82 126.746 0)
+			(hide yes)
+			(show_name no)
+			(do_not_autoplace no)
+			(effects
+				(font
+					(size 1.27 1.27)
+				)
+				(justify bottom)
+			)
+		)
+		(property "CREATOR" "NEZY"
+			(at 83.82 126.746 0)
+			(hide yes)
+			(show_name no)
+			(do_not_autoplace no)
+			(effects
+				(font
+					(size 1.27 1.27)
+				)
+				(justify bottom)
+			)
+		)
+		(property "Price" "None"
+			(at 83.82 126.746 0)
+			(hide yes)
+			(show_name no)
+			(do_not_autoplace no)
+			(effects
+				(font
+					(size 1.27 1.27)
+				)
+				(justify bottom)
+			)
+		)
+		(property "Package" "WQFN-24 Texas Instruments"
+			(at 83.82 126.746 0)
+			(hide yes)
+			(show_name no)
+			(do_not_autoplace no)
+			(effects
+				(font
+					(size 1.27 1.27)
+				)
+				(justify bottom)
+			)
+		)
+		(property "Check_prices" "https://www.snapeda.com/parts/BQ25896RTWR/Texas+Instruments/view-part/?ref=eda"
+			(at 89.408 125.73 0)
+			(hide yes)
+			(show_name no)
+			(do_not_autoplace no)
+			(effects
+				(font
+					(size 1.27 1.27)
+				)
+				(justify bottom)
+			)
+		)
+		(property "STANDARD" "Manufacturer Recommendations"
+			(at 83.82 126.746 0)
+			(hide yes)
+			(show_name no)
+			(do_not_autoplace no)
+			(effects
+				(font
+					(size 1.27 1.27)
+				)
+				(justify bottom)
+			)
+		)
+		(property "PARTREV" "C"
+			(at 83.82 126.746 0)
+			(hide yes)
+			(show_name no)
+			(do_not_autoplace no)
+			(effects
+				(font
+					(size 1.27 1.27)
+				)
+				(justify bottom)
+			)
+		)
+		(property "VERIFIER" ""
 			(at 97.79 85.09 0)
 			(hide yes)
@@
 					(size 1.27 1.27)
 				)
-			)
-		)
-		(pin "37"
-		)
-		(pin "39"
-		)
-		(pin "38"
-		)
-		(pin "45"
-		)
-		(pin "40"
-		)
-		(pin "41"
-		)
-		(pin "43"
-		)
-		(pin "42"
-		)
-		(pin "44"
-		)
-		(pin "57"
-		)
-		(pin "55"
-		)
-		(pin "61"
-		)
-		(pin "51"
-		)
-		(pin "47"
-		)
-		(pin "50"
-		)
-		(pin "46"
-		)
-		(pin "64"
-		)
-		(pin "63"
-		)
-		(pin "59"
-		)
-		(pin "52"
-		)
-		(pin "56"
-		)
-		(pin "49"
-		)
-		(pin "58"
-		)
-		(pin "60"
-		)
-		(pin "62"
-		)
-		(pin "54"
-		)
-		(pin "53"
-		)
-		(pin "48"
+				(justify bottom)
+			)
+		)
+		(property "SnapEDA_Link" "https://www.snapeda.com/parts/BQ25896RTWR/Texas+Instruments/view-part/?ref=snap"
+			(at 89.408 125.73 0)
+			(hide yes)
+			(show_name no)
+			(do_not_autoplace no)
+			(effects
+				(font
+					(size 1.27 1.27)
+				)
+				(justify bottom)
+			)
+		)
+		(property "MP" "BQ25896RTWR"
+			(at 83.82 126.746 0)
+			(hide yes)
+			(show_name no)
+			(do_not_autoplace no)
+			(effects
+				(font
+					(size 1.27 1.27)
+				)
+				(justify bottom)
+			)
+		)
+		(property "Availability" "In Stock"
+			(at 83.82 126.746 0)
+			(hide yes)
+			(show_name no)
+			(do_not_autoplace no)
+			(effects
+				(font
+					(size 1.27 1.27)
+				)
+				(justify bottom)
+			)
+		)
+		(property "MANUFACTURER" "Texas Instruments"
+			(at 83.82 126.746 0)
+			(hide yes)
+			(show_name no)
+			(do_not_autoplace no)
+			(effects
+				(font
+					(size 1.27 1.27)
+				)
+				(justify bottom)
+			)
 		)
 		(pin "3"
@@
 		)
 		(pin "25"
-		)
-		(pin "27"
-		)
-		(pin "30"
-		)
-		(pin "35"
-		)
-		(pin "36"
-		)
-		(pin "34"
-		)
-		(pin "26"
-		)
-		(pin "33"
-		)
-		(pin "28"
-		)
-		(pin "32"
-		)
-		(pin "29"
-		)
-		(pin "31"
 		)
 		(instances
@@
 					(reference "U2")
 					(unit 1)
+				)
+				(path "/158d6e2c-2f49-4796-8b5c-460e7c4b776f/6335dc05-b9de-40bf-a572-b195fb20e3fd"
+					(reference "U2")
+					(unit 1)
