File: Garbage_collector_pcb/STM32.kicad_sch (KiCad schematic)
At the start: 18 parts, among them J1 Conn_ST_STDC14, J10 NRF52840, SW1 SW_Push, U1 STM32G431RBTx, Y2 24MHz

Commit message: finalisation des empreintes
Parts:
- J1: renamed from J10; footprint Connector_JST:JST_GH_BM03B-GHS-TBT_1x03-1MP_P1.25mm_Vertical -> Connector_JST:JST_GH_BM04B-GHS-TBT_1x04-1MP_P1.25mm_Vertical
- R1: renamed from R3; footprint Resistor_THT:R_Array_SIP4 -> Resistor_SMD:R_0402_1005Metric
- SW1: footprint (none) -> Button_Switch_SMD:SW_Push_1P1T_NO_CK_KMR2
- renumbered C12 to C10, C13 to C11, C14 to C12, C4 to C3, C6 to C4, C7 to C5, C8 to C6, C9 to C7, C10 to C8, C11 to C9, J1 to J2, Y2 to Y1
Changed lines of the file:
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@@
 		(dnp no)
 		(fields_autoplaced yes)
-		(property "Reference" "C4"
+		(property "Reference" "C3"
 			(at 55.88 69.8499 0)
 			(show_name no)
@@
 			(project "Garbage_collector"
 				(path "/158d6e2c-2f49-4796-8b5c-460e7c4b776f/06023c4c-7891-4ab0-97ab-4f54be3e219b"
-					(reference "C4")
+					(reference "C3")
 					(unit 1)
 				)
@@
 		(dnp no)
 		(fields_autoplaced yes)
-		(property "Reference" "C11"
+		(property "Reference" "C9"
 			(at 137.16 25.4062 0)
 			(show_name no)
@@
 			(project "Garbage_collector"
 				(path "/158d6e2c-2f49-4796-8b5c-460e7c4b776f/06023c4c-7891-4ab0-97ab-4f54be3e219b"
-					(reference "C11")
+					(reference "C9")
 					(unit 1)
 				)
@@
 		(dnp no)
 		(fields_autoplaced yes)
-		(property "Reference" "#FLG05"
+		(property "Reference" "#FLG01"
 			(at 258.445 40.64 0)
 			(hide yes)
@@
 			(project "Garbage_collector"
 				(path "/158d6e2c-2f49-4796-8b5c-460e7c4b776f/06023c4c-7891-4ab0-97ab-4f54be3e219b"
-					(reference "#FLG05")
+					(reference "#FLG01")
 					(unit 1)
 				)
@@
 		(dnp no)
 		(fields_autoplaced yes)
-		(property "Reference" "J1"
+		(property "Reference" "J2"
 			(at 265.43 60.9599 0)
 			(show_name no)
@@
 			(project "Garbage_collector"
 				(path "/158d6e2c-2f49-4796-8b5c-460e7c4b776f/06023c4c-7891-4ab0-97ab-4f54be3e219b"
-					(reference "J1")
+					(reference "J2")
 					(unit 1)
 				)
@@
 			)
 		)
-		(property "Footprint" ""
+		(property "Footprint" "Button_Switch_SMD:SW_Push_1P1T_NO_CK_KMR2"
 			(at 25.4 48.26 0)
 			(hide yes)
@@
 		(dnp no)
 		(fields_autoplaced yes)
-		(property "Reference" "#PWR065"
+		(property "Reference" "#PWR010"
 			(at 231.14 146.05 0)
 			(hide yes)
@@
 			(project "Garbage_collector"
 				(path "/158d6e2c-2f49-4796-8b5c-460e7c4b776f/06023c4c-7891-4ab0-97ab-4f54be3e219b"
-					(reference "#PWR065")
+					(reference "#PWR010")
 					(unit 1)
 				)
@@
 		(dnp no)
 		(fields_autoplaced yes)
-		(property "Reference" "Y2"
+		(property "Reference" "Y1"
 			(at 52.07 63.4999 90)
 			(show_name no)
@@
 			(project "Garbage_collector"
 				(path "/158d6e2c-2f49-4796-8b5c-460e7c4b776f/06023c4c-7891-4ab0-97ab-4f54be3e219b"
-					(reference "Y2")
+					(reference "Y1")
 					(unit 1)
 				)
@@
 		(dnp no)
 		(fields_autoplaced yes)
-		(property "Reference" "C9"
+		(property "Reference" "C7"
 			(at 118.11 25.4062 0)
 			(show_name no)
@@
 			(project "Garbage_collector"
 				(path "/158d6e2c-2f49-4796-8b5c-460e7c4b776f/06023c4c-7891-4ab0-97ab-4f54be3e219b"
-					(reference "C9")
+					(reference "C7")
 					(unit 1)
 				)
@@
 		(dnp no)
 		(fields_autoplaced yes)
-		(property "Reference" "C12"
+		(property "Reference" "C10"
 			(at 147.32 25.4062 0)
 			(show_name no)
@@
 			(project "Garbage_collector"
 				(path "/158d6e2c-2f49-4796-8b5c-460e7c4b776f/06023c4c-7891-4ab0-97ab-4f54be3e219b"
-					(reference "C12")
+					(reference "C10")
 					(unit 1)
 				)
@@
 		(in_pos_files yes)
 		(dnp no)
-		(property "Reference" "C7"
+		(property "Reference" "C5"
 			(at 66.04 41.91 0)
 			(show_name no)
@@
 			(project "Garbage_collector"
 				(path "/158d6e2c-2f49-4796-8b5c-460e7c4b776f/06023c4c-7891-4ab0-97ab-4f54be3e219b"
-					(reference "C7")
+					(reference "C5")
 					(unit 1)
 				)
@@
 		(dnp no)
 		(fields_autoplaced yes)
-		(property "Reference" "#PWR02"
+		(property "Reference" "#PWR03"
 			(at 38.1 82.55 0)
 			(hide yes)
@@
 			(project "Garbage_collector"
 				(path "/158d6e2c-2f49-4796-8b5c-460e7c4b776f/06023c4c-7891-4ab0-97ab-4f54be3e219b"
-					(reference "#PWR02")
+					(reference "#PWR03")
 					(unit 1)
 				)
@@
 		(in_pos_files yes)
 		(dnp no)
-		(property "Reference" "C6"
+		(property "Reference" "C4"
 			(at 57.912 41.656 0)
 			(show_name no)
@@
 			(project "Garbage_collector"
 				(path "/158d6e2c-2f49-4796-8b5c-460e7c4b776f/06023c4c-7891-4ab0-97ab-4f54be3e219b"
-					(reference "C6")
+					(reference "C4")
 					(unit 1)
 				)
@@
 		(dnp no)
 		(fields_autoplaced yes)
-		(property "Reference" "#PWR07"
+		(property "Reference" "#PWR06"
 			(at 99.06 144.78 0)
 			(hide yes)
@@
 			(project "Garbage_collector"
 				(path "/158d6e2c-2f49-4796-8b5c-460e7c4b776f/06023c4c-7891-4ab0-97ab-4f54be3e219b"
-					(reference "#PWR07")
+					(reference "#PWR06")
 					(unit 1)
 				)
@@
 		(dnp no)
 		(fields_autoplaced yes)
-		(property "Reference" "#PWR01"
+		(property "Reference" "#PWR02"
 			(at 31.75 69.85 0)
 			(hide yes)
@@
 			(project "Garbage_collector"
 				(path "/158d6e2c-2f49-4796-8b5c-460e7c4b776f/06023c4c-7891-4ab0-97ab-4f54be3e219b"
-					(reference "#PWR01")
+					(reference "#PWR02")
 					(unit 1)
 				)
@@
 		(dnp no)
 		(fields_autoplaced yes)
-		(property "Reference" "#PWR09"
+		(property "Reference" "#PWR08"
 			(at 105.41 39.37 0)
 			(hide yes)
@@
 			(project "Garbage_collector"
 				(path "/158d6e2c-2f49-4796-8b5c-460e7c4b776f/06023c4c-7891-4ab0-97ab-4f54be3e219b"
-					(reference "#PWR09")
+					(reference "#PWR08")
 					(unit 1)
 				)
@@
 		(in_pos_files yes)
 		(dnp no)
-		(property "Reference" "#PWR092"
+		(property "Reference" "#PWR04"
 			(at 58.42 40.64 0)
 			(hide yes)
@@
 			(project "Garbage_collector"
 				(path "/158d6e2c-2f49-4796-8b5c-460e7c4b776f/06023c4c-7891-4ab0-97ab-4f54be3e219b"
-					(reference "#PWR092")
+					(reference "#PWR04")
 					(unit 1)
 				)
@@
 		(dnp no)
 		(fields_autoplaced yes)
-		(property "Reference" "#FLG010"
+		(property "Reference" "#FLG02"
 			(at 258.445 81.28 0)
 			(hide yes)
@@
 			(project "Garbage_collector"
 				(path "/158d6e2c-2f49-4796-8b5c-460e7c4b776f/06023c4c-7891-4ab0-97ab-4f54be3e219b"
-					(reference "#FLG010")
+					(reference "#FLG02")
 					(unit 1)
 				)
@@
 		(dnp no)
 		(fields_autoplaced yes)
-		(property "Reference" "#PWR06"
+		(property "Reference" "#PWR05"
 			(at 58.42 55.88 0)
 			(hide yes)
@@
 			(project "Garbage_collector"
 				(path "/158d6e2c-2f49-4796-8b5c-460e7c4b776f/06023c4c-7891-4ab0-97ab-4f54be3e219b"
-					(reference "#PWR06")
+					(reference "#PWR05")
 					(unit 1)
 				)
@@
 		(dnp no)
 		(fields_autoplaced yes)
-		(property "Reference" "R3"
+		(property "Reference" "R1"
 			(at 66.04 62.2299 0)
 			(show_name no)
@@
 			)
 		)
-		(property "Footprint" "Resistor_THT:R_Array_SIP4"
+		(property "Footprint" "Resistor_SMD:R_0402_1005Metric"
 			(at 62.23 63.5 0)
 			(hide yes)
@@
 			(project "Garbage_collector"
 				(path "/158d6e2c-2f49-4796-8b5c-460e7c4b776f/06023c4c-7891-4ab0-97ab-4f54be3e219b"
-					(reference "R3")
+					(reference "R1")
 					(unit 1)
 				)
@@
 		(dnp no)
 		(fields_autoplaced yes)
-		(property "Reference" "C10"
+		(property "Reference" "C8"
 			(at 128.27 25.4062 0)
 			(show_name no)
@@
 			(project "Garbage_collector"
 				(path "/158d6e2c-2f49-4796-8b5c-460e7c4b776f/06023c4c-7891-4ab0-97ab-4f54be3e219b"
-					(reference "C10")
+					(reference "C8")
 					(unit 1)
 				)
@@
 		(in_pos_files yes)
 		(dnp no)
-		(property "Reference" "#PWR093"
+		(property "Reference" "#PWR09"
 			(at 231.14 133.35 0)
 			(hide yes)
@@
 			(project "Garbage_collector"
 				(path "/158d6e2c-2f49-4796-8b5c-460e7c4b776f/06023c4c-7891-4ab0-97ab-4f54be3e219b"
-					(reference "#PWR093")
+					(reference "#PWR09")
 					(unit 1)
 				)
@@
 		(dnp no)
 		(fields_autoplaced yes)
-		(property "Reference" "C14"
+		(property "Reference" "C12"
 			(at 166.37 25.4062 0)
 			(show_name no)
@@
 			(project "Garbage_collector"
 				(path "/158d6e2c-2f49-4796-8b5c-460e7c4b776f/06023c4c-7891-4ab0-97ab-4f54be3e219b"
-					(reference "C14")
+					(reference "C12")
 					(unit 1)
 				)
@@
 		(dnp no)
 		(fields_autoplaced yes)
-		(property "Reference" "C8"
+		(property "Reference" "C6"
 			(at 107.95 25.4062 0)
 			(show_name no)
@@
 			(project "Garbage_collector"
 				(path "/158d6e2c-2f49-4796-8b5c-460e7c4b776f/06023c4c-7891-4ab0-97ab-4f54be3e219b"
-					(reference "C8")
+					(reference "C6")
 					(unit 1)
 				)
@@
 		(dnp no)
 		(fields_autoplaced yes)
-		(property "Reference" "C13"
+		(property "Reference" "C11"
 			(at 157.48 25.4062 0)
 			(show_name no)
@@
 			(project "Garbage_collector"
 				(path "/158d6e2c-2f49-4796-8b5c-460e7c4b776f/06023c4c-7891-4ab0-97ab-4f54be3e219b"
-					(reference "C13")
+					(reference "C11")
 					(unit 1)
 				)
@@
 		(dnp no)
 		(fields_autoplaced yes)
-		(property "Reference" "J10"
+		(property "Reference" "J1"
 			(at 240.03 133.3499 0)
 			(show_name no)
@@
 			)
 		)
-		(property "Footprint" "Connector_JST:JST_GH_BM03B-GHS-TBT_1x03-1MP_P1.25mm_Vertical"
+		(property "Footprint" "Connector_JST:JST_GH_BM04B-GHS-TBT_1x04-1MP_P1.25mm_Vertical"
 			(at 237.49 133.35 0)
 			(hide yes)
@@
 			(project "Garbage_collector"
 				(path "/158d6e2c-2f49-4796-8b5c-460e7c4b776f/06023c4c-7891-4ab0-97ab-4f54be3e219b"
-					(reference "J10")
+					(reference "J1")
 					(unit 1)
 				)
@@
 		(dnp no)
 		(fields_autoplaced yes)
-		(property "Reference" "#PWR08"
+		(property "Reference" "#PWR07"
 			(at 105.41 24.13 0)
 			(hide yes)
@@
 			(project "Garbage_collector"
 				(path "/158d6e2c-2f49-4796-8b5c-460e7c4b776f/06023c4c-7891-4ab0-97ab-4f54be3e219b"
-					(reference "#PWR08")
+					(reference "#PWR07")
 					(unit 1)
 				)

Commit message: fin du routage
Parts:
- C1: JLCPCB Part # C32949 -> C1525
- C12: JLCPCB Part # C52923 -> C29266
- C2, C3: value 20pF -> 10pF; JLCPCB Part # C32949 -> 32949
- C4: JLCPCB Part # C14445 -> C29266
- J1: JLCPCB Part # (none) -> C161692
- Y1: value 24MHz -> 16MHz
Connections:
- net CHARGEUR_PG renamed Chargeur_OTG
Changed lines of the file:
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@@
 		)
 	)
-	(hierarchical_label "CHARGEUR_PG"
+	(hierarchical_label "Chargeur_OTG"
 		(shape input)
 		(at 115.57 104.14 0)
@@
 			)
 		)
-		(property "Value" "20pF"
+		(property "Value" "10pF"
 			(at 55.88 72.3899 0)
 			(show_name no)
@@
 			)
 		)
-		(property "JLCPCB Part #" "C32949"
+		(property "JLCPCB Part #" "32949"
 			(at 53.34 71.12 0)
 			(hide yes)
@@
 			)
 		)
-		(property "Value" "24MHz"
+		(property "Value" "16MHz"
 			(at 52.07 66.0399 90)
 			(show_name no)
@@
 			)
 		)
-		(property "Value" "20pF"
+		(property "Value" "10pF"
 			(at 40.64 72.3899 0)
 			(show_name no)
@@
 			)
 		)
-		(property "JLCPCB Part #" "C32949"
+		(property "JLCPCB Part #" "32949"
 			(at 38.1 71.12 0)
 			(hide yes)
@@
 			)
 		)
-		(property "JLCPCB Part #" "C14445"
+		(property "JLCPCB Part #" "C29266"
 			(at 54.61 43.18 0)
 			(hide yes)
@@
 			)
 		)
-		(property "JLCPCB Part #" "C32949"
+		(property "JLCPCB Part #" "C1525"
 			(at 31.75 58.42 0)
 			(hide yes)
@@
 			)
 		)
-		(property "JLCPCB Part #" "C52923"
+		(property "JLCPCB Part #" "C29266"
 			(at 163.83 26.67 0)
 			(hide yes)
@@
 			(at 237.49 133.35 0)
 			(hide yes)
+			(show_name no)
+			(do_not_autoplace no)
+			(effects
+				(font
+					(size 1.27 1.27)
+				)
+			)
+		)
+		(property "JLCPCB Part #" "C161692"
+			(at 237.49 133.35 0)
+			(hide yes)

Commit message: generation du gerber, fichier de perçage, BOM et PCL pour la commande
Parts:
- C2, C3: JLCPCB Part # 32949 -> C32949
Changed lines of the file:
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@@
 			)
 		)
-		(property "JLCPCB Part #" "32949"
+		(property "JLCPCB Part #" "C32949"
 			(at 53.34 71.12 0)
 			(hide yes)
@@
 			)
 		)
-		(property "JLCPCB Part #" "32949"
+		(property "JLCPCB Part #" "C32949"
 			(at 38.1 71.12 0)
 			(hide yes)
