File: Garbage_collector_pcb/Alim.kicad_sch (KiCad schematic)
At the start: 62 parts, among them J2 USB_C_Receptacle_PowerOnly_6P, J4 NEOPIXELS, Q1 MMDT2907A-7-F, Q2 DMP1045U-7, Q3 DMN313DLT-7, SW2 SW_Push, U2 BQ27220YZFR, U3 BQ25896RTWR, U6 SN74AHCT1G125DBVR

Commit message: ajout du ioc et schema validé
Parts:
- removed C31: 100n, Capacitor_SMD:C_0402_1005Metric, symbol Device:C_Small
- removed F1: 250 mA, Fuse:Fuse_0603_1608Metric, symbol Device:Polyfuse_Small
- removed FB1: 120Ω@100MHz, Inductor_SMD:L_0603_1608Metric, symbol Device:FerriteBead
- removed J4: NEOPIXELS, Connector_JST:JST_GH_SM03B-GHS-TB_1x03-1MP_P1.25mm_Horizontal, symbol Connector_Generic:Conn_01x03
- removed R12: 300, Resistor_SMD:R_0603_1608Metric, symbol Device:R_Small
- removed U6: SN74AHCT1G125DBVR, Package_TO_SOT_SMD:SOT-23-5, symbol 74xGxx:74AHCT1G125
- added JP5: SolderJumper_2_Open, Jumper:SolderJumper-2_P1.3mm_Open_TrianglePad1.0x1.5mm, symbol Jumper:SolderJumper_2_Open
- added TP5, TP6: TestPoint, TestPoint:TestPoint_Pad_D2.0mm, symbol Connector:TestPoint
- C15, C18, C19: value 1µ -> 1u; footprint (none) -> Capacitor_SMD:C_0402_1005Metric
- C20, C25, C28, C35, C36, C38: footprint (none) -> Capacitor_SMD:C_0402_1005Metric
- D3: value LED -> LEG_ROUGE
- D4: value LED -> LED_VERTE
- D5: value LED -> LED_JAUNE
- D6: value LED -> LED_BLEUE
- R9: value 0.01 -> 10m
- SW2: JLCPCB Part # (none) -> C72443; JLCPCB Part# C72443 -> (none)
Connections:
- net +5V: no longer JP4.2 (B)
- net +BATT: no longer C15.2, PS1.1 (VIN), PS1.3 (STBY)
- net EXP: now also TP5.1
- net SYS: now also C15.2, PS1.1 (VIN), PS1.3 (STBY), JP5.2 (B), TP6.1; no longer C35.1, C36.1, L1.1, TP4.1, U3.15 (SYS), U3.16 (SYS)
- net VBUS: now also J2.A9 (VBUS), J2.B9 (VBUS), JP4.2 (B); no longer Q1.4 (E2), Q2.3 (D)
- net VBUS_BQ25: now reaches Q1.1 (E1), Q2.2 (S), TP3.1
- net VBUS_BQ25: now also C18.2, JP3.2 (B), U3.1 (VBUS); no longer JP4.1 (A)
- net CHARGEUR_QON: now reaches C37.2, SW2.1, U3.12 (~{QON})
- net GPOUT renamed FG_GPIO
- net INT renamed CHARGEUR_INT
- net ~{PG} renamed CHARGEUR_PG
- new net: C35.1, C36.1, JP5.1 (A), L1.1, TP4.1, U3.15 (SYS), U3.16 (SYS)
- new net: JP4.1 (A), Q1.4 (E2), Q2.3 (D)
Other:
- note removed: "NEOPIXELS RING"
- moved on the sheet: C15, C19, D3, D4, D5, D6, JP4, L1, PS1, R17, R18, R19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
