File: Garbage_collector_pcb/Alim.kicad_sch (KiCad schematic)
At the start: 59 parts, among them J2 USB_C_Receptacle_PowerOnly_6P, Q1 MMDT2907A-7-F, Q2 DMP1045U-7, Q3 DMN313DLT-7, SW2 SW_Push, U2 BQ27220YZFR, U3 BQ25896RTWR

Commit message: finalisation des empreintes
Parts:
- BT1: footprint (none) -> Connector_JST:JST_GH_SM02B-GHS-TB_1x02-1MP_P1.25mm_Horizontal
- D1: renamed from D3; footprint (none) -> LED_SMD:LED_0603_1608Metric
- D2: renamed from D4; footprint (none) -> LED_SMD:LED_0603_1608Metric
- D3: renamed from D5; footprint (none) -> LED_SMD:LED_0603_1608Metric
- D4: renamed from D6; footprint (none) -> LED_SMD:LED_0603_1608Metric
- J3: renamed from J2; footprint (none) -> Connector_USB:USB_C_Receptacle_GCT_USB4125-xx-x-0190_6P_TopMnt_Horizontal
- R10: renamed from R13; footprint (none) -> Resistor_SMD:R_0402_1005Metric
- R12: renamed from R19; footprint (none) -> Resistor_SMD:R_0402_1005Metric
- R15: renamed from R22; footprint (none) -> Resistor_SMD:R_0402_1005Metric
- R20: renamed from R25; footprint (none) -> Resistor_SMD:R_0402_1005Metric
- R23: renamed from R26; footprint (none) -> Resistor_SMD:R_0402_1005Metric
- SW2: footprint (none) -> Button_Switch_SMD:SW_Push_1P1T_NO_CK_KMR2
- renumbered C15 to C13, C39 to C14, C40 to C15, C19 to C16, C20 to C17, C38 to C19, C21 to C20, C25 to C21, C28 to C22, C35 to C23, C37 to C24, C23 to C25, C36 to C26, JP3 to JP1, JP4 to JP2, JP5 to JP3, R34 to R11, R35 to R13, R20 to R14, R32 to R16, R21 to R19, R5 to R2, R23 to R21, R24 to R22, R6 to R3, R7 to R4, R8 to R5, R9 to R6, R10 to R7, R11 to R8, R33 to R9, TP6 to TP1, TP1 to TP3, TP5 to TP4, TP3 to TP5, TP4 to TP6

Commit message: routage du pcb quasiment terminé, 1 erreur DRC
Parts:
- U2: footprint Package_BGA:Texas_DSBGA-9_1.4715x1.4715mm_Layout3x3_P0.5mm -> Package_BGA:Texas_DSBGA-9_1.62x1.58mm_Layout3x3_P0.5mm
Changed lines of the file:
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@@
 			)
 		)
-		(property "Footprint" "Package_BGA:Texas_DSBGA-9_1.4715x1.4715mm_Layout3x3_P0.5mm"
+		(property "Footprint" "Package_BGA:Texas_DSBGA-9_1.62x1.58mm_Layout3x3_P0.5mm"
 			(at 33.02 135.89 0)
 			(hide yes)

Commit message: fin du routage
Parts:
- removed R17: 10k, Resistor_SMD:R_0402_1005Metric, symbol Device:R_Small
- C15: JLCPCB Part # C72203 -> C12530
- C25: JLCPCB Part # C318563 -> C23733
- D1: JLCPCB Part # (none) -> C2286; JLCPCB Part# (none) -> C2286
- D2: JLCPCB Part # (none) -> C99289; JLCPCB Part# (none) -> C99289
- D3: value LED_JAUNE -> LED_ORANGE; JLCPCB Part # (none) -> C84269; JLCPCB Part# (none) -> C84269
- D4: value LED_BLEUE -> LED_ROUGE; JLCPCB Part # (none) -> C2286; JLCPCB Part# (none) -> C2286
- R12, R23: value 100k -> 1k; JLCPCB Part # (none) -> C11702; JLCPCB Part# (none) -> C11702
- R15, R20: value 100k -> 2k2; JLCPCB Part # (none) -> C25879; JLCPCB Part# (none) -> C25879
Connections:
- net CHARGEUR_PG renamed Chargeur_PG
- net OTG renamed Chargeur_OTG
Other:
- moved on the sheet: R18

Commit message: generation du gerber, fichier de perçage, BOM et PCL pour la commande
Parts:
- J3: JLCPCB Part # C2927026 -> C963366
- TP1, TP2, TP3, TP4, TP5, TP6: now left out of the parts list
Changed lines of the file:
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@@
 		(body_style 1)
 		(exclude_from_sim no)
-		(in_bom yes)
+		(in_bom no)
 		(on_board yes)
 		(in_pos_files yes)
@@
 		(body_style 1)
 		(exclude_from_sim no)
-		(in_bom yes)
+		(in_bom no)
 		(on_board yes)
 		(in_pos_files yes)
@@
 		(body_style 1)
 		(exclude_from_sim no)
-		(in_bom yes)
+		(in_bom no)
 		(on_board yes)
 		(in_pos_files yes)
@@
 		(body_style 1)
 		(exclude_from_sim no)
-		(in_bom yes)
+		(in_bom no)
 		(on_board yes)
 		(in_pos_files yes)
@@
 		(body_style 1)
 		(exclude_from_sim no)
-		(in_bom yes)
+		(in_bom no)
 		(on_board yes)
 		(in_pos_files yes)
@@
 		(body_style 1)
 		(exclude_from_sim no)
-		(in_bom yes)
+		(in_bom no)
 		(on_board yes)
 		(in_pos_files yes)
@@
 			)
 		)
-		(property "JLCPCB Part #" "C2927026"
+		(property "JLCPCB Part #" "C963366"
 			(at 27.94 35.56 0)
 			(hide yes)
