File: Garbage_collector_pcb/Moteurs.kicad_sch (KiCad schematic)
At the start: 16 parts, among them J4 MOTOR2, J5 MOTOR1, J6 SERVO1, J7 SERVO2, U4 DRV8833PWP

Commit message: fin du routage
Parts:
- C28: JLCPCB Part # C76614 -> C70225
- C29: JLCPCB Part # (none) -> C96180
Changed lines of the file:
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@@
 			)
 		)
-		(property "JLCPCB Part #" "C76614"
+		(property "JLCPCB Part #" "C70225"
 			(at 73.66 69.85 0)
 			(hide yes)
@@
 			(at 80.01 69.85 0)
 			(hide yes)
+			(show_name no)
+			(do_not_autoplace no)
+			(effects
+				(font
+					(size 1.27 1.27)
+				)
+			)
+		)
+		(property "JLCPCB Part #" "C96180"
+			(at 80.01 69.85 0)
+			(hide yes)
