File: Garbage_collector_pcb/Capteurs.kicad_sch (KiCad schematic)
At the start: 14 parts, among them J10 Lidar, J11 VL53L0CXV0DH1, J12 NEOPIXELS, J8 VL53L0CXV0DH1, J9 ADA3595, U5 SN74AHCT1G125DBVR

Commit message: fin du routage
Parts:
- J10: JLCPCB Part # (none) -> C161692
Changed lines of the file:
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@@
+			)
+		)
+		(property "JLCPCB Part #" "C161692"
+			(at 68.58 81.28 0)
+			(hide yes)
+			(show_name no)
+			(do_not_autoplace no)
+			(effects
+				(font
+					(size 1.27 1.27)
+				)
 			)
 		)

Commit message: generation du gerber, fichier de perçage, BOM et PCL pour la commande
Parts:
- R27, R28: footprint Resistor_SMD:R_0603_1608Metric_Pad0.98x0.95mm_HandSolder -> Resistor_SMD:R_0402_1005Metric; now left out of the parts list
Changed lines of the file:
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@@
 		(body_style 1)
 		(exclude_from_sim no)
-		(in_bom yes)
+		(in_bom no)
 		(on_board yes)
 		(in_pos_files yes)
@@
 			)
 		)
-		(property "Footprint" "Resistor_SMD:R_0603_1608Metric_Pad0.98x0.95mm_HandSolder"
+		(property "Footprint" "Resistor_SMD:R_0402_1005Metric"
 			(at 144.78 34.29 0)
 			(hide yes)
@@
 		(body_style 1)
 		(exclude_from_sim no)
-		(in_bom yes)
+		(in_bom no)
 		(on_board yes)
 		(in_pos_files yes)
@@
 			)
 		)
-		(property "Footprint" "Resistor_SMD:R_0603_1608Metric_Pad0.98x0.95mm_HandSolder"
+		(property "Footprint" "Resistor_SMD:R_0402_1005Metric"
 			(at 123.19 34.29 0)
 			(hide yes)
