File: Garbage_collector_pcb/Garbage_collector.kicad_pcb (KiCad board)
At the start: 4 copper layers, 86.9 x 52.9 mm, 110 parts, among them J1 NRF52840, J10 Lidar, J11 VL53L0CXV0DH1, J12 NEOPIXELS, J2 Conn_ST_STDC14, J3 USB_C_Receptacle_PowerOnly_6P, J4 MOTOR2, J5 MOTOR1, J6 SERVO1, J7 SERVO2, J8 VL53L0CXV0DH1, J9 ADA3595, Q1 MMDT2907A-7-F, Q2 DMP1045U-7, Q3 DMN313DLT-7, SW1 SW_Push, SW2 SW_Push, U1 STM32G431RBTx, U2 BQ27220YZFR, U3 BQ25896RTWR, U4 DRV8833PWP, U5 SN74AHCT1G125DBVR, Y1 16MHz

Commit message: generation du gerber, fichier de perçage, BOM et PCL pour la commande
Parts:
- D3: value LED_JAUNE -> LED_ORANGE
- D4: value LED_BLEUE -> LED_ROUGE
- R12, R23: value 100k -> 1k
- R15, R20: value 100k -> 2k2
- R27, R28: footprint Resistor_SMD:R_0603_1608Metric_Pad0.98x0.95mm_HandSolder -> Resistor_SMD:R_0402_1005Metric
Routing:
- net Net-(JP3-A): track 16.8 -> 17.1 mm, vias 0 -> 1
- net /Moteurs/BOUT2: vias 4 -> 0
- net /Moteurs/BOUT1: vias 3 -> 0
- net /Moteurs/AOUT2: vias 3 -> 0
- net /Moteurs/AOUT1: vias 3 -> 0
- added copper zone on F.Cu, net Net-(JP3-A)
Other:
- board text added: "QON"
- board text added: "RST"
